File: portail_moteur_continu.kicad_pcb (KiCad board)
At the start: 2 copper layers, 140 x 80 mm, 84 parts, among them J1 Screw_Terminal_01x02, J10 Conn_01x01_Male, J11 Conn_01x08_Male, J2 Screw_Terminal_01x03, J3 Conn_01x04, J4 Screw_Terminal_01x06, J5 Screw_Terminal_01x03, J6 Conn_01x06_Male, J7 Screw_Terminal_01x02, J8 Conn_01x01_Male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

Commit message: V1.1
Parts:
- moved FID7 1.00 mm to (164.5, 54.0)
- moved FID8 1.00 mm to (202.0, 102.5)
- moved J4 0.90 mm to (229.4, 101.5)
- moved K1 0.89 mm to (214.7, 127.3)
Routing:
- net /SDA: track 98.6 -> 95.7 mm, vias 2 -> 1
- net /SCL: track 100.4 -> 97.5 mm, vias 2 -> 1
- net Net-(J4-Pad4): track 26.9 -> 25.7 mm
- net Net-(J4-Pad3): track 7.47 -> 6.58 mm
- net Net-(J4-Pad2): track 7.50 -> 6.61 mm
- net Net-(J4-Pad1): track 7.54 -> 6.65 mm
- net Net-(C1-Pad2): track 27.1 -> 28.0 mm
- net Net-(J4-Pad6): track 23.4 -> 23.9 mm

Commit message: maj 10-09-22
Parts:
- removed R25, R27: 1k, Resistor_THT:R_Axial_DIN0207_L6.3mm_D2.5mm_P7.62mm_Horizontal
- added D7: 1N4004, Diode_THT:D_DO-41_SOD81_P10.16mm_Horizontal, F.Cu at (194.9, 122.5)
- added R18: 5k, Resistor_THT:R_Axial_DIN0207_L6.3mm_D2.5mm_P7.62mm_Horizontal, F.Cu at (130.1, 103.7)
- added R24: 1k, Resistor_THT:R_Axial_DIN0207_L6.3mm_D2.5mm_P7.62mm_Horizontal, F.Cu at (109.5, 112.1)
- added R26: 5k, Resistor_THT:R_Axial_DIN0207_L6.3mm_D2.5mm_P7.62mm_Horizontal, F.Cu at (122.5, 100.5)
- added R32: 1k, Resistor_THT:R_Axial_DIN0207_L6.3mm_D2.5mm_P7.62mm_Horizontal, F.Cu at (132.5, 100.5)
- moved R8 4.59 mm to (122.5, 106.9)
Connections:
- A1 pad 27: +5V -> Net-(A1-Pad27)
Routing:
- net /PRIS: track 72.8 -> 107.8 mm
- net /PLIS: track 79.6 -> 98.4 mm
- net /RIS: track 14.6 -> 21.6 mm
- net +5V: track 364.1 -> 370.4 mm
- net Net-(A1-Pad27): track 0.00 -> 3.42 mm
- net /LIS: track 39.5 -> 38.0 mm
- net Net-(R8-Pad2): track 21.7 -> 23.0 mm
- net /FOuv: track 47.2 -> 47.9 mm
Other:
- board text added: "F1IWQ sept 2022"
- board text added: "https://github.com/f1iwq2/Belfox_IWQ"
